File: RCC.kicad_pcb (KiCad board)
At the start: 4 copper layers, 44.5 x 37 mm, 45 parts, among them J1 Battery, J2 USB_C_Receptacle_USB2.0_16P, J3 Conn_01x07, J4 Conn_01x04_Pin, SW2 SW_Push, U1 BQ24040DGQR, U2 ESD7104MUTAG, U3 TLV75801PDRV, U5 STM32L412KBTx, Y1 ECS-2520MVQ-480-CN-TR

Commit message: Restructure folder and start revB
Parts:
- removed C13: 1uF, Capacitor_SMD:C_0603_1608Metric
- removed G***: LOGO, LOGO
- removed SW2: SW_Push, Button_Switch_SMD:SW_Push_1P1T_NO_CK_KMR2
- removed U5: STM32L412KBTx, Package_QFP:LQFP-32_7x7mm_P0.8mm
- removed Y1: ECS-2520MVQ-480-CN-TR, ECS_2520MVQ_480_CN_TR:OSC_ECS-2520S25-250-FN-TR
- added C17: 10nF, Capacitor_SMD:C_0603_1608Metric, F.Cu at (161.8, 79.1)
- added R12: 0, Resistor_SMD:R_0603_1608Metric, F.Cu at (169.8, 81.6)
- added R2: 1M, Resistor_SMD:R_0603_1608Metric, F.Cu at (165.8, 71.6)
- added R3: 1k, Resistor_SMD:R_0603_1608Metric, F.Cu at (165.8, 74.1)
- added SW1: SW_Push, Button_Switch_SMD:SW_Push_1P1T_NO_CK_KMR2, F.Cu at (167.2, 96.6)
- added TP1: TestPoint, TestPoint:TestPoint_Pad_D1.0mm, F.Cu at (159.3, 84.4)
- added TP2: TestPoint, TestPoint:TestPoint_Pad_D1.0mm, F.Cu at (159.3, 87.5)
- added TP3: TestPoint, TestPoint:TestPoint_Pad_D1.0mm, F.Cu at (159.3, 90.5)
- added TP4: TestPoint, TestPoint:TestPoint_Pad_D1.0mm, F.Cu at (133.0, 97.5)
- added TP5: TestPoint, TestPoint:TestPoint_Pad_D1.0mm, F.Cu at (162.3, 84.4)
- added TP6: TestPoint, TestPoint:TestPoint_Pad_D1.0mm, F.Cu at (162.3, 87.5)
- added TP7: TestPoint, TestPoint:TestPoint_Pad_D1.0mm, F.Cu at (162.3, 90.5)
- added U4: STM32L412KBTx, Package_QFP:LQFP-32_7x7mm_P0.8mm, F.Cu at (122.2, 83.5)
- C10: value 10uF -> 1uF
- C11: value 10nF -> 1uF; moved to F.Cu
- C12: value 1uF -> 0.1uF; moved to F.Cu
- C14, C15, FB1: moved to F.Cu
- C16: value 0.1uF -> 2.2uF
- C2, C7: value 1uF -> 0.1uF
- C3: value 0.1uF -> 1uF
- C4: value 2.2uF -> 1uF
- C5: value 10nF -> 1uF
- C6: value 1uF -> 10uF
- C9: value 0.1uF -> 10nF
- D1: value LED_Small -> Charging
- D2: value BC_Status -> LED_Small
- D3: value Charging -> BC_Status
- H1, H2, H3, H4: footprint MountingHole:MountingHole_3.2mm_M3 -> MountingHole:MountingHole_2.2mm_M2
- J1: footprint Connector_JST:JST_PH_S2B-PH-K_1x02_P2.00mm_Horizontal -> Connector_JST:JST_PH_S2B-PH-SM4-TB_1x02-1MP_P2.00mm_Horizontal; moved to B.Cu
- R10, R9: value 1k -> 0
- R4: value 1M -> 200k
- R5: value 200k -> 1k
- R6: value 10k -> 1k; moved to F.Cu
- R8: value 1k -> 10k
- U1: value BQ24040DGQR -> TLV75801PDRV; footprint BQ24040DSQR:SON40P200X200X80-11N -> Package_SON:WSON-6-1EP_2x2mm_P0.65mm_EP1x1.6mm
- U2: value ESD7104MUTAG -> BQ24040DGQR; footprint ESD7104:UDFN10_ONS -> BQ24040DSQR:SON40P200X200X80-11N
- U3: value TLV75801PDRV -> USBLC6-2SC6; footprint Package_SON:WSON-6-1EP_2x2mm_P0.65mm_EP1x1.6mm -> USBLC6_2SC6:SOT95P280X145-6N
- moved D1 60.1 mm to (177.3, 84.2), turned to 0 degrees
- moved U3 55.8 mm to (173.7, 96.5)
- moved R8 53.2 mm to (169.8, 71.6), turned to 0 degrees
- moved C16 48.6 mm to (161.8, 76.6), turned to 0 degrees
- moved R4 47.9 mm to (165.8, 76.6)
- moved FB1 46.6 mm to (161.8, 81.6), turned to 0 degrees
- moved R5 46.3 mm to (165.8, 79.1)
- moved D4 45.7 mm to (177.3, 92.0)
- moved D3 45.7 mm to (177.3, 89.4), turned to 0 degrees
- moved D2 44.4 mm to (177.3, 86.8), turned to 0 degrees
- moved U1 44.0 mm to (173.9, 77.1), turned to 0 degrees
- moved U2 44.0 mm to (174.4, 73.5), turned to 0 degrees
- moved C14 43.7 mm to (161.8, 71.6), turned to 0 degrees
- moved C12 43.6 mm to (157.8, 81.6), turned to 0 degrees
- moved R6 43.6 mm to (165.8, 81.6), turned to 0 degrees
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- renumbered J3 to J2, J2 to J3
Connections:
- C10 pad 1: +3V3 -> +3.3VA
- C11 pad 1: +3.3VA -> +3V3
- C12 pad 1: +3.3VA -> /NRST
- C14 pad 1: /NRST -> /SW_BOOT0
- C15 pad 1: /SW_BOOT0 -> GND
- C15 pad 2: GND -> +3V3
- C16 pad 1: +3V3 -> GND
- C16 pad 2: GND -> +3V3
- C2 pad 1: /VBAT -> /VBUS
- C3 pad 1: GND -> +3V3
- C3 pad 2: +3V3 -> GND
- C4 pad 1: GND -> /VBAT
- C4 pad 2: +3V3 -> GND
- C5 pad 1: GND -> /VBAT
- C5 pad 2: +3V3 -> GND
- C6 pad 1: /VBAT -> +3V3
- C9 pad 1: +3V3 -> +3.3VA
- D1 pad 1: GND -> /CHG_STATUS
- D2 pad 1: Net-(D2-K) -> GND
- D3 pad 1: /CHG_STATUS -> Net-(D3-K)
- MT1 pad 1: /MISO -> Net-(MT1-AP_SDO/AP_AD0)
- R1 pad 1: Net-(U1-ISET) -> /VBAT
- R1 pad 2: GND -> Net-(D1-A)
- R10 pad 1: /VBAT -> Net-(U4-PA7)
- R10 pad 2: Net-(D3-A) -> /MOSI
- R4 pad 1: +3V3 -> Net-(U1-FB)
- R4 pad 2: Net-(U3-FB) -> GND
- R5 pad 1: Net-(U3-FB) -> Net-(U2-ISET)
- R6 pad 1: /SW_BOOT0 -> /VBAT
- R6 pad 2: /BOOT0 -> Net-(D3-A)
- R8 pad 1: +3V3 -> /SW_BOOT0
- R8 pad 2: Net-(D1-A) -> /BOOT0
- R9 pad 1: /VBAT -> Net-(U4-PA5)
- R9 pad 2: Net-(D2-A) -> /SCLK
- U1 pad 1: /VBUS -> +3V3
- U1 pad 2: Net-(U1-ISET) -> Net-(U1-FB)
- U1 pad 4: unconnected-(U1-PRETERM-Pad4) -> /VBAT
- U1 pad 5: Net-(D2-K) -> unconnected-(U1-DNC-Pad5)
- U1 pad 6: (no net) -> /VBAT
- U2 pad 1: /USB_N -> /VBUS
- U2 pad 10: /USB_N -> /VBAT
- U2 pad 2: /USB_P -> Net-(U2-ISET)
- U2 pad 5: /VBUS -> Net-(D3-K)
- U2 pad 6: /VBUS -> (no net)
- U2 pad 7: unconnected-(U2-NC-Pad7) -> GND
- U2 pad 8: GND -> /CHG_STATUS
- U2 pad 9: /USB_P -> unconnected-(U2-TS-Pad9)
- U3 pad 1: +3V3 -> /USB_N
- U3 pad 2: Net-(U3-FB) -> GND
- U3 pad 3: GND -> /USB_P
- U3 pad 4: /VBAT -> /USB_P
- U3 pad 5: unconnected-(U3-DNC-Pad5) -> /VBUS
- U3 pad 6: /VBAT -> /USB_N
Routing:
- net +3V3: track 99.9 -> 0.00 mm, vias 2 -> 0
- net GND: track 61.0 -> 0.00 mm, vias 23 -> 0
- net /SCLK: track 27.9 -> 0.00 mm, vias 2 -> 0
- net /MOSI: track 27.2 -> 0.00 mm, vias 1 -> 0
- net /VBAT: track 21.6 -> 0.00 mm
- net /VBUS: track 19.6 -> 0.00 mm
- net /DIS_CS: track 18.2 -> 0.00 mm, vias 1 -> 0
- net /CHG_STATUS: track 16.1 -> 0.00 mm, vias 2 -> 0
- net /SWCLK: track 14.4 -> 0.00 mm, vias 1 -> 0
- net /SWDIO: track 13.8 -> 0.00 mm, vias 1 -> 0
- net /DIS_RST: track 13.2 -> 0.10 mm, vias 1 -> 0
- net +3.3VA: track 13.1 -> 0.00 mm, vias 1 -> 0
- net /DIS_DC: track 13.7 -> 0.65 mm, vias 1 -> 0
- net /USB_N: track 12.9 -> 0.00 mm
- net /USB_P: track 12.8 -> 0.00 mm
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Other:
- board text removed: "3V3"
- board text removed: "BATTERY"
- board text removed: "BOOT"
- board text removed: "BoJoe"
- board text removed: "CHG"
- board text removed: "DEBUG"
- board text removed: "DISPLAY"
- board text removed: "Dashi"
- board text removed: "GYRO"
- board text removed: "POW"
- board text removed: "USB"
- board text removed: "blinky"
- board text removed: "daa"

Commit message: Finish routing revB
Parts:
- removed R11: 1k, Resistor_SMD:R_0603_1608Metric
- removed TP6, TP7: TestPoint, TestPoint:TestPoint_Pad_D1.0mm
- added R13: 5k1, Resistor_SMD:R_0603_1608Metric, F.Cu at (133.5, 91.3)
- added R14: 5k1, Resistor_SMD:R_0603_1608Metric, F.Cu at (132.0, 82.5)
- added R15: 0, Resistor_SMD:R_0603_1608Metric, F.Cu at (121.5, 94.2)
- added R7: 1k, Resistor_SMD:R_0603_1608Metric, F.Cu at (111.8, 73.0)
- C10: value 1uF -> 10nF
- C12, C2: value 0.1uF -> 1uF
- C5: value 1uF -> 10uF
- C6: value 10uF -> 0.1uF
- C9: value 10nF -> 0.1uF
- D1: value Charging -> BC_Status
- D2: value LED_Small -> Charging
- D3: value BC_Status -> power_status
- J1: footprint Connector_JST:JST_PH_S2B-PH-SM4-TB_1x02-1MP_P2.00mm_Horizontal -> Connector_JST:JST_PH_S2B-PH-K_1x02_P2.00mm_Horizontal; moved to F.Cu
- J2: value Conn_01x07 -> DEBUG HEADER; footprint Connector_JST:JST_PH_S7B-PH-K_1x07_P2.00mm_Horizontal -> Connector_JST:JST_PH_S4B-PH-K_1x04_P2.00mm_Horizontal
- J4: value Conn_01x04_Pin -> DISPLAY_HEADER; footprint Connector_JST:JST_PH_S4B-PH-K_1x04_P2.00mm_Horizontal -> Connector_PinSocket_2.54mm:PinSocket_1x07_P2.54mm_Vertical
- R12: value 0 -> 1k
- R2: value 1M -> 1k
- R3: value 1k -> 10k
- R4: value 200k -> 1k
- R5: value 1k -> 1M
- R6: value 1k -> 200k
- SW1: footprint Button_Switch_SMD:SW_Push_1P1T_NO_CK_KMR2 -> EVQPUA02K:KEY-SMD_EVQPUAXXX
- TP1, TP2, TP3, TP4, TP5: moved to B.Cu
- U1: value TLV75801PDRV -> BQ24040DGQR; footprint Package_SON:WSON-6-1EP_2x2mm_P0.65mm_EP1x1.6mm -> BQ24040DSQR:SON40P200X200X80-11N
- U2: value BQ24040DGQR -> TLV75801PDRV; footprint BQ24040DSQR:SON40P200X200X80-11N -> Package_SON:WSON-6-1EP_2x2mm_P0.65mm_EP1x1.6mm
- U3: value USBLC6-2SC6 -> STM32L412KBTx; footprint USBLC6_2SC6:SOT95P280X145-6N -> Package_QFP:LQFP-32_7x7mm_P0.8mm
- U4: value STM32L412KBTx -> USBLC6-2SC6; footprint Package_QFP:LQFP-32_7x7mm_P0.8mm -> USBLC6_2SC6:SOT95P280X145-6N
- moved D3 68.1 mm to (111.8, 70.8), turned to 180 degrees
- moved U2 65.9 mm to (108.8, 79.1), turned to 180 degrees
- moved D4 65.1 mm to (115.8, 70.8)
- moved R8 60.2 mm to (113.5, 92.8)
- moved R12 54.8 mm to (115.8, 73.0), turned to 180 degrees
- moved R5 54.4 mm to (111.5, 82.8), turned to 90 degrees
- moved R6 54.4 mm to (111.5, 79.2), turned to 90 degrees
- moved U3 54.1 mm to (121.1, 84.0)
- moved FB1 53.5 mm to (108.5, 86.0)
- moved R9 53.3 mm to (119.3, 91.2), turned to -90 degrees
- moved SW1 51.4 mm to (115.8, 98.0)
- moved C7 51.1 mm to (113.5, 94.5), turned to 180 degrees
- moved D2 51.0 mm to (128.8, 71.0), turned to 180 degrees
- moved R10 50.2 mm to (121.8, 91.2), turned to -90 degrees
- moved C10 49.6 mm to (109.8, 89.0), turned to -90 degrees
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Connections:
- C1 pad 2: /VBUS -> /USB Connector/VBUS
- C11 pad 1: +3V3 -> +3.3VA
- C12 pad 1: /NRST -> +3V3
- C14 pad 1: /SW_BOOT0 -> GND
- C14 pad 2: GND -> /USB Connector/VBUS
- C17 pad 1: GND -> +3V3
- C17 pad 2: +3V3 -> GND
- C2 pad 1: /VBUS -> /Battery Charger/VOUT
- C3 pad 1: +3V3 -> /Battery Charger/VOUT
- C4 pad 1: /VBAT -> +3V3
- C5 pad 1: /VBAT -> +3V3
- C6 pad 1: +3V3 -> /Microcontroller/NRST
- C7 pad 1: +3V3 -> /Microcontroller/SW_BOOT0
- C9 pad 1: +3.3VA -> +3V3
- D1 pad 1: /CHG_STATUS -> /Battery Charger/PG_N
- D2 pad 1: GND -> /Battery Charger/CHG_N
- D3 pad 1: Net-(D3-K) -> GND
- J1 pad 1: /VBAT -> /Battery Charger/VOUT
- J2 pad 2: GND -> /Microcontroller/SWDIO
- J2 pad 3: /MOSI -> /Microcontroller/SWCLK
- J2 pad 4: /SCLK -> GND
- J3 pad A4: /VBUS -> /USB Connector/VBUS
- J3 pad A5: unconnected-(J3-CC1-PadA5) -> /USB Connector/CC1
- J3 pad A6: /USB_P -> /USB Connector/USB_P
- J3 pad A7: /USB_N -> /USB Connector/USB_N
- J3 pad A9: /VBUS -> /USB Connector/VBUS
- J3 pad B4: /VBUS -> /USB Connector/VBUS
- J3 pad B5: unconnected-(J3-CC2-PadB5) -> /USB Connector/CC2
- J3 pad B6: /USB_P -> /USB Connector/USB_P
- J3 pad B7: /USB_N -> /USB Connector/USB_N
- J3 pad B9: /VBUS -> /USB Connector/VBUS
- J4 pad 2: /SWDIO -> GND
- J4 pad 3: /SWCLK -> /Gyroscope and Accelerometer/MISO
- J4 pad 4: GND -> /Gyroscope and Accelerometer/SCLK
- MT1 pad 1: Net-(MT1-AP_SDO/AP_AD0) -> /Gyroscope and Accelerometer/GMISO
- MT1 pad 12: /GYRO_CS -> /Gyroscope and Accelerometer/GYRO_CS
- MT1 pad 13: /SCLK -> /Gyroscope and Accelerometer/SCLK
- MT1 pad 14: /MOSI -> /Gyroscope and Accelerometer/MOSI
- MT1 pad 4: /GY_INT1 -> /Gyroscope and Accelerometer/GY_INT1
- MT1 pad 9: /GY_INT2 -> /Gyroscope and Accelerometer/GY_INT2
- R1 pad 1: /VBAT -> /Battery Charger/ISET
- R1 pad 2: Net-(D1-A) -> GND
- R10 pad 1: Net-(U4-PA7) -> /Microcontroller/MMOSI
- R10 pad 2: /MOSI -> /Gyroscope and Accelerometer/MOSI
- R12 pad 1: /MISO -> Net-(D4-A)
- R12 pad 2: Net-(MT1-AP_SDO/AP_AD0) -> /Microcontroller/TEST_LED
- R2 pad 1: +3V3 -> /Battery Charger/VOUT
- R2 pad 2: Net-(U1-FB) -> Net-(D1-A)
- R3 pad 1: +3V3 -> /Battery Charger/TS
- R3 pad 2: Net-(D2-A) -> GND
- R4 pad 1: Net-(U1-FB) -> /Battery Charger/VOUT
- R4 pad 2: GND -> Net-(D2-A)
- R5 pad 1: Net-(U2-ISET) -> +3V3
- R5 pad 2: GND -> /Voltage Regulator/FB
- R6 pad 1: /VBAT -> /Voltage Regulator/FB
- R6 pad 2: Net-(D3-A) -> GND
- R8 pad 1: /SW_BOOT0 -> /Microcontroller/SW_BOOT0
- R8 pad 2: /BOOT0 -> /Microcontroller/BOOT0
- R9 pad 1: Net-(U4-PA5) -> /Microcontroller/MSCLK
- R9 pad 2: /SCLK -> /Gyroscope and Accelerometer/SCLK
- SW1 pad 1: /SW_BOOT0 -> +3V3
- SW1 pad 2: +3V3 -> /Microcontroller/SW_BOOT0
- TP1 pad 1: /VBAT -> /Gyroscope and Accelerometer/MOSI
- TP2 pad 1: /GY_INT1 -> /Gyroscope and Accelerometer/MISO
- TP3 pad 1: /GY_INT2 -> /Microcontroller/BOOT0
- TP4 pad 1: /GYRO_CS -> +3V3
- TP5 pad 1: /SCLK -> GND
- U1 pad 1: +3V3 -> /USB Connector/VBUS
- U1 pad 2: Net-(U1-FB) -> /Battery Charger/ISET
- U1 pad 4: /VBAT -> unconnected-(U1-PRETERM-Pad4)
- U1 pad 5: unconnected-(U1-DNC-Pad5) -> /Battery Charger/PG_N
- U1 pad 6: /VBAT -> (no net)
- U2 pad 1: /VBUS -> +3V3
- U2 pad 2: Net-(U2-ISET) -> /Voltage Regulator/FB
- U2 pad 4: unconnected-(U2-PRETERM-Pad4) -> /Battery Charger/VOUT
- U2 pad 5: Net-(D3-K) -> unconnected-(U2-DNC-Pad5)
- U2 pad 6: (no net) -> /Battery Charger/VOUT
- U3 pad 1: /USB_N -> +3V3
- U3 pad 2: GND -> unconnected-(U3-PC14-Pad2)
- U3 pad 3: /USB_P -> unconnected-(U3-PC15-Pad3)
- U3 pad 4: /USB_P -> /Microcontroller/NRST
- U3 pad 5: /VBUS -> +3.3VA
- U3 pad 6: /USB_N -> unconnected-(U3-PA0-Pad6)
- U4 pad 1: +3V3 -> /USB Connector/USB_N
- U4 pad 2: unconnected-(U4-PC14-Pad2) -> GND
- U4 pad 3: unconnected-(U4-PC15-Pad3) -> /USB Connector/USB_P
- U4 pad 4: /NRST -> /USB Connector/USB_P
- U4 pad 5: +3.3VA -> /USB Connector/VBUS
- U4 pad 6: /HSE_IN -> /USB Connector/USB_N
Routing:
- net +3V3: track 0.00 -> 104.1 mm, vias 0 -> 2
- net GND: track 0.00 -> 51.5 mm, vias 0 -> 43
- net /Battery Charger/VOUT: track 0.00 -> 41.2 mm
- net /Gyroscope and Accelerometer/SCLK: track 0.00 -> 31.7 mm, vias 0 -> 2
- net /Gyroscope and Accelerometer/MISO: track 0.00 -> 30.3 mm, vias 0 -> 1
- net /Microcontroller/BOOT0: track 0.00 -> 30.0 mm, vias 0 -> 2
- net /USB Connector/VBUS: track 0.00 -> 26.1 mm
- net /Microcontroller/DIS_RST: track 0.00 -> 18.0 mm, vias 0 -> 1
- net /Battery Charger/CHG_N: track 0.00 -> 17.5 mm, vias 0 -> 3
- net /Microcontroller/DIS_DC: track 0.00 -> 16.1 mm, vias 0 -> 1
- net /Microcontroller/DIS_CS: track 0.00 -> 15.6 mm, vias 0 -> 1
- net /Microcontroller/SWCLK: track 0.00 -> 14.9 mm, vias 0 -> 1
- net /Microcontroller/SWDIO: track 0.00 -> 14.8 mm, vias 0 -> 1
- net /USB Connector/USB_N: track 0.00 -> 14.7 mm
- net /USB Connector/USB_P: track 0.00 -> 14.0 mm
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Other:
- outline, holes or cut-outs redrawn
- board text added: "+"
- board text added: "-"
- board text added: "3V3"
- board text added: "BLK"
- board text added: "BOOT0"
- board text added: "CHG"
- board text added: "CLK"
- board text added: "CS"
- board text added: "DC"
- board text added: "DIN"
- board text added: "GND"
- board text added: "MISO"
- board text added: "MOSI"
- board text added: "POW"
- board text added: "RST"
- board text added: "SWCLK"
- board text added: "SWDIO"

Commit message: Add silkscreen to pcb
Parts:
- added G***: LOGO, LOGO, F.Cu at (107.7, 96.1)
Other:
- board text added: "By BoJoe"
- board text added: "Dashidaaa"
- board text added: "x"
- board text added: "y"
- board text added: "z"
