File: RCC.kicad_pcb (KiCad board)
At the start: 4 copper layers, 44.5 x 37 mm, 55 parts, among them J1 Battery, J2 DEBUG HEADER, J3 USB_C_Receptacle_USB2.0_16P, J4 DISPLAY_HEADER, SW1 SW_Push, U1 BQ24040DGQR, U2 TLV75801PDRV, U3 STM32L412KBTx, U4 USBLC6-2SC6

Commit message: Finnish RevB
Parts:
- removed R3: 10k, Resistor_SMD:R_0603_1608Metric
- C1, C10, C11, C12, C14, C15, C16, C17, C2, C3, C4, C5: footprint Capacitor_SMD:C_0603_1608Metric -> Capacitor_SMD:C_0603_1608Metric_Pad1.08x0.95mm_HandSolder
- C6, C7, C8, C9: footprint Capacitor_SMD:C_0603_1608Metric -> Capacitor_SMD:C_0402_1005Metric_Pad0.74x0.62mm_HandSolder
- D1, D2, D3, D4: footprint LED_SMD:LED_0603_1608Metric -> LED_SMD:LED_0603_1608Metric_Pad1.05x0.95mm_HandSolder
- FB1: value 120R -> 600R; footprint Inductor_SMD:L_0603_1608Metric -> Inductor_SMD:L_0603_1608Metric_Pad1.05x0.95mm_HandSolder
- R1, R10, R12, R13, R14, R15, R2, R4, R5, R6, R7, R8, R9: footprint Resistor_SMD:R_0603_1608Metric -> Resistor_SMD:R_0603_1608Metric_Pad0.98x0.95mm_HandSolder
- SW1: value SW_Push -> ~; footprint EVQPUA02K:KEY-SMD_EVQPUAXXX -> SW-SMD_TS24CA:SW-SMD_TS24CA
- U3: value STM32L412KBTx -> STM32L432KBUx; footprint Package_QFP:LQFP-32_7x7mm_P0.8mm -> Package_DFN_QFN:QFN-32-1EP_5x5mm_P0.5mm_EP3.45x3.45mm
- moved TP2 3.67 mm to (122.2, 88.2)
- moved C8 3.07 mm to (117.4, 81.5)
- moved C5 2.93 mm to (115.4, 81.4)
- moved C9 2.28 mm to (125.2, 86.8)
- moved R1 1.74 mm to (132.8, 76.7)
- moved U1 1.74 mm to (129.8, 77.6)
- moved C11 1.63 mm to (113.3, 88.5)
- moved C10 1.53 mm to (111.2, 88.5)
- moved C6 1.49 mm to (116.1, 83.8), turned to 180 degrees
- moved C2 1.36 mm to (128.2, 79.7)
- moved C1 1.29 mm to (132.2, 79.8)
- moved C12 0.81 mm to (109.2, 84.1)
- moved C4 0.81 mm to (109.5, 81.4)
- moved FB1 0.81 mm to (109.2, 85.8)
- moved R5 0.81 mm to (112.3, 82.6)
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Connections:
- SW1 pad 1: +3V3 -> unconnected-(SW1-Pad1)
- SW1 pad 3: (no net) -> +3V3
- SW1 pad 4: (no net) -> unconnected-(SW1-Pad4)
- U1 pad 9: /Battery Charger/TS -> unconnected-(U1-TS-Pad9)
Routing:
- net /Microcontroller/BOOT0: track 30.0 -> 37.9 mm, vias 2 -> 4
- net /Gyroscope and Accelerometer/MISO: track 30.3 -> 35.9 mm
- net GND: track 51.5 -> 56.0 mm, vias 43 -> 45
- net /Battery Charger/VOUT: track 41.2 -> 44.8 mm
- net +3V3: track 104.1 -> 100.8 mm, vias 2 -> 3
- net /USB Connector/USB_N: track 14.7 -> 17.8 mm
- net /USB Connector/USB_P: track 14.0 -> 16.9 mm
- net +3.3VA: track 11.8 -> 14.7 mm
- net /Battery Charger/TS: track 2.58 -> 0.00 mm
- net /Microcontroller/SWCLK: track 14.9 -> 17.2 mm
- net /Gyroscope and Accelerometer/GY_INT1: track 12.8 -> 14.8 mm
- net /Gyroscope and Accelerometer/GY_INT2: track 8.22 -> 10.2 mm
- net /Gyroscope and Accelerometer/GYRO_CS: track 6.63 -> 8.48 mm
- net /Gyroscope and Accelerometer/SCLK: track 31.7 -> 33.4 mm
- net /Microcontroller/SWDIO: track 14.8 -> 16.5 mm
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