File: RCC.kicad_sch (KiCad schematic)
At the start: 50 parts, among them J1 Battery, J2 USB_C_Receptacle_USB2.0_16P, J3 Conn_01x07, J4 Conn_01x04_Pin, SW2 SW_Push, U1 BQ24040DGQR, U3 TLV75801PDRV, U4 USBLC6-2SC6, U5 STM32L412KBTx, Y1 ECS-2520MVQ-480-CN-TR

Commit message: Restructure folder and start revB
Parts:
- removed R7: 1k5, Resistor_SMD:R_0603_1608Metric, symbol Device:R_Small
- added TP1, TP2, TP3, TP4, TP5, TP6, TP7: TestPoint, TestPoint:TestPoint_Pad_D1.0mm, symbol Connector:TestPoint
- C13: renamed from C16; now not fitted
- H1, H2, H3, H4: footprint MountingHole:MountingHole_3.2mm_M3 -> MountingHole:MountingHole_2.2mm_M2
- J1: footprint Connector_JST:JST_PH_S2B-PH-K_1x02_P2.00mm_Horizontal -> Connector_JST:JST_PH_S2B-PH-SM4-TB_1x02-1MP_P2.00mm_Horizontal
- R7: renamed from R2; now not fitted
- U3: renamed from U4; footprint USBLC6-2SC6:SOT95P280X145-6N -> USBLC6_2SC6:SOT95P280X145-6N
- Y1: now not fitted
- renumbered C12 to C10, C13 to C11, C14 to C12, C15 to C14, C3 to C15, C4 to C16, C5 to C17, C17 to C2, C7 to C3, C6 to C4, C2 to C5, C10 to C6, C9 to C7, C11 to C9, D3 to D1, D1 to D2, D2 to D3, J3 to J2, J2 to J3, R10 to R1, R12 to R10, R13 to R12, R4 to R2, R8 to R3, R5 to R4, R1 to R5, R9 to R6, R6 to R8, R3 to R9, SW2 to SW1, U3 to U1, U1 to U2, U5 to U4
Connections:
- net GYRO_CS: now also TP4.1
- net GY_INT1: now also TP2.1
- net GY_INT2: now also TP3.1
- net MISO: now also TP6.1
- net MOSI: now also TP7.1
- net SCLK: now also TP5.1
- net VBAT: now also TP1.1
Other:
- note added: "Display mount are M2 Display dimension: 44.5mm x 37mm"
- note removed: "AN4879 Application notes"
- note removed: "Display mount are M3 Display dimension: 44.5mm x 37mm"
- moved on the sheet: C2, C5

Commit message: Finish routing revB
Parts:
- removed C1, C10, C11, C3, C4, C5: 1uF, Capacitor_SMD:C_0603_1608Metric, symbol Device:C_Small
- removed C12, C13, C14, C15, C2, C7, C8: 0.1uF, Capacitor_SMD:C_0603_1608Metric, symbol Device:C_Small
- removed C16: 2.2uF, Capacitor_SMD:C_0603_1608Metric, symbol Device:C_Small
- removed C17, C9: 10nF, Capacitor_SMD:C_0603_1608Metric, symbol Device:C_Small
- removed C6: 10uF, Capacitor_SMD:C_0603_1608Metric, symbol Device:C_Small
- removed D1: Charging, LED_SMD:LED_0603_1608Metric, symbol Device:LED_Small
- removed D2, D4: LED_Small, LED_SMD:LED_0603_1608Metric, symbol Device:LED_Small
- removed D3: BC_Status, LED_SMD:LED_0603_1608Metric, symbol Device:LED_Small
- removed FB1: 120R, Inductor_SMD:L_0603_1608Metric, symbol Device:FerriteBead_Small
- removed J2: Conn_01x07, Connector_JST:JST_PH_S7B-PH-K_1x07_P2.00mm_Horizontal, symbol Connector_Generic:Conn_01x07
- removed J3: USB_C_Receptacle_USB2.0_16P, Connector_USB:USB_C_Receptacle_G-Switch_GT-USB-7010ASV, symbol Connector:USB_C_Receptacle_USB2.0_16P
- removed J4: Conn_01x04_Pin, Connector_JST:JST_PH_S4B-PH-K_1x04_P2.00mm_Horizontal, symbol Connector:Conn_01x04_Pin
- removed MT1: ICM-42670-P, ICM42670:XDCR_ICM-42670-P, symbol ICM-42670-P:ICM-42670-P
- removed R1, R11, R3, R5, R6: 1k, Resistor_SMD:R_0603_1608Metric, symbol Device:R_Small
- removed R10, R12, R7, R9: 0, Resistor_SMD:R_0603_1608Metric, symbol Device:R_Small
- removed R2: 1M, Resistor_SMD:R_0603_1608Metric, symbol Device:R_Small
- removed R4: 200k, Resistor_SMD:R_0603_1608Metric, symbol Device:R_Small
- removed R8: 10k, Resistor_SMD:R_0603_1608Metric, symbol Device:R_Small
- removed SW1: SW_Push, Button_Switch_SMD:SW_Push_1P1T_NO_CK_KMR2, symbol Switch:SW_Push
- removed TP1, TP2, TP3, TP4, TP5, TP6, TP7: TestPoint, TestPoint:TestPoint_Pad_D1.0mm, symbol Connector:TestPoint
- removed U1: TLV75801PDRV, Package_SON:WSON-6-1EP_2x2mm_P0.65mm_EP1x1.6mm, symbol Regulator_Linear:TLV75801PDRV
- removed U2: BQ24040DGQR, BQ24040DSQR:SON40P200X200X80-11N, symbol BQ24040DGQR:BQ24040DGQR
- removed U3: USBLC6-2SC6, USBLC6_2SC6:SOT95P280X145-6N, symbol USBLC6-2SC6:USBLC6-2SC6
- removed U4: STM32L412KBTx, Package_QFP:LQFP-32_7x7mm_P0.8mm, symbol MCU_ST_STM32L4:STM32L412KBTx
- removed Y1: ECS-2520MVQ-480-CN-TR, ECS_2520MVQ_480_CN_TR:OSC_ECS-2520S25-250-FN-TR, symbol ECS-2520MVQ-480-CN-TR:ECS-2520MVQ-480-CN-TR
- J1: footprint Connector_JST:JST_PH_S2B-PH-SM4-TB_1x02-1MP_P2.00mm_Horizontal -> Connector_JST:JST_PH_S2B-PH-K_1x02_P2.00mm_Horizontal
Connections:
- net VBAT renamed Battery Charger/VOUT
- no-connect marks 17 -> 0
Other:
- added sheet Battery Charger (battery_charger.kicad_sch)
- added sheet Gyroscope and Accelerometer (gyro_accel.kicad_sch)
- added sheet Microcontroller (microcontroller.kicad_sch)
- added sheet Oled RGB Display (display.kicad_sch)
- added sheet USB Connector (usb_connector.kicad_sch)
- added sheet Voltage Regulator (voltage_regulator.kicad_sch)
- note removed: "Notes: - write command when DATA/COMMAND (DC) = 0, write data when DC = 1 - DIS_CS is active low"
- note removed: "VOUT = VFB × (1 + R1 / R2), VFB = 0.55V R1 + R2 ≤ VOUT / (IFB × 100),IFB = 10 nA R1/R2 = 5 R1 + R2 ≤ 3300000"
- moved on the sheet: H1, H2, H3, H4, J1

Commit message: Finnish RevB
Other:
- note added: "note: using JLC04161H-3313 Stackup"
- moved on the sheet: J1
