File: microcontroller.kicad_sch (KiCad schematic)
At the start: 18 parts, among them J2 DEBUG HEADER, SW1 SW_Push, U3 STM32L412KBTx

Commit message: Add silkscreen to pcb
Changed lines of the file:
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@@
+	)
+	(junction
+		(at 152.4 74.93)
+		(diameter 0)
+		(color 0 0 0 0)
 	)
 	(junction
@@
 	)
 	(junction
-		(at 147.32 74.93)
-		(diameter 0)
-		(color 0 0 0 0)
-	)
-	(junction
 		(at 114.3 73.66)
 		(diameter 0)
@@
 	(wire
 		(pts
+			(xy 152.4 74.93) (xy 149.86 74.93)
+		)
+		(stroke
+			(width 0)
+			(type default)
+		)
+	)
+	(wire
+		(pts
 			(xy 153.67 104.14) (xy 160.02 104.14)
 		)
@@
 	(wire
 		(pts
-			(xy 147.32 74.93) (xy 149.86 74.93)
-		)
-		(stroke
-			(width 0)
-			(type default)
-		)
-	)
-	(wire
-		(pts
 			(xy 167.64 74.93) (xy 176.53 74.93)
 		)
@@
 	(wire
 		(pts
-			(xy 143.51 74.93) (xy 147.32 74.93)
+			(xy 143.51 74.93) (xy 149.86 74.93)
 		)
 		(stroke
@@
 	(wire
 		(pts
-			(xy 149.86 74.93) (xy 160.02 74.93)
-		)
-		(stroke
-			(width 0)
-			(type default)
-		)
-	)
-	(wire
-		(pts
 			(xy 153.67 93.98) (xy 158.75 93.98)
 		)
@@
 		(pts
 			(xy 138.43 73.66) (xy 138.43 82.55)
+		)
+		(stroke
+			(width 0)
+			(type default)
+		)
+	)
+	(wire
+		(pts
+			(xy 152.4 74.93) (xy 160.02 74.93)
 		)
 		(stroke
@@
 	(symbol
 		(lib_id "power:PWR_FLAG")
-		(at 147.32 74.93 0)
+		(at 152.4 74.93 0)
 		(unit 1)
 		(exclude_from_sim no)
@@
 		(dnp no)
 		(property "Reference" "#FLG01"
-			(at 147.32 73.025 0)
+			(at 152.4 73.025 0)
 			(effects
 				(font
@@
 		)
 		(property "Value" "PWR_FLAG"
-			(at 150.368 70.866 0)
+			(at 155.448 70.866 0)
 			(effects
 				(font
@@
 		)
 		(property "Footprint" ""
-			(at 147.32 74.93 0)
+			(at 152.4 74.93 0)
 			(effects
 				(font
@@
 		)
 		(property "Datasheet" "~"
-			(at 147.32 74.93 0)
+			(at 152.4 74.93 0)
 			(effects
 				(font
@@
 		)
 		(property "Description" "Special symbol for telling ERC where power comes from"
-			(at 147.32 74.93 0)
-			(effects
-				(font
+			(at 152.4 74.93 0)
+			(effects
+				(font

Commit message: Finnish RevB
Parts:
- removed SW1: SW_Push, EVQPUA02K:KEY-SMD_EVQPUAXXX, symbol Switch:SW_Push
- removed U3: STM32L412KBTx, Package_QFP:LQFP-32_7x7mm_P0.8mm, symbol MCU_ST_STM32L4:STM32L412KBTx
- added SW1: ~, SW-SMD_TS24CA:SW-SMD_TS24CA, symbol SW-SMD_TS24CA:TS24CA
- added U3: STM32L432KBUx, Package_DFN_QFN:QFN-32-1EP_5x5mm_P0.5mm_EP3.45x3.45mm, symbol MCU_ST_STM32L4:STM32L432KBUx
- C10, C11, C12, C5: footprint Capacitor_SMD:C_0603_1608Metric -> Capacitor_SMD:C_0603_1608Metric_Pad1.08x0.95mm_HandSolder
- C6, C7, C8, C9: footprint Capacitor_SMD:C_0603_1608Metric -> Capacitor_SMD:C_0402_1005Metric_Pad0.74x0.62mm_HandSolder
- D4: footprint LED_SMD:LED_0603_1608Metric -> LED_SMD:LED_0603_1608Metric_Pad1.05x0.95mm_HandSolder
- FB1: value 120R -> 600R; footprint Inductor_SMD:L_0603_1608Metric -> Inductor_SMD:L_0603_1608Metric_Pad1.05x0.95mm_HandSolder
- R10, R12, R8, R9: footprint Resistor_SMD:R_0603_1608Metric -> Resistor_SMD:R_0603_1608Metric_Pad0.98x0.95mm_HandSolder
Connections:
- net +3.3VA: now also U3.5 (VDDA)
- net +3V3: now also SW1.3, U3.1 (VDD), U3.17 (VDD)
- net BOOT0: now also U3.31 (PH3)
- net CHG_N: now also U3.27 (PB4)
- net DIS_CS: now also U3.7 (PA1)
- net DIS_DC: now also U3.8 (PA2)
- net DIS_RST: now also U3.9 (PA3)
- net GND: now also U3.16 (VSS), U3.32 (VSS), U3.33 (VSS)
- net GYRO_CS: now also U3.14 (PB0)
- net GY_INT1: now also U3.10 (PA4)
- net GY_INT2: now also U3.15 (PB1)
- net MISO: now also U3.12 (PA6)
- net MMOSI: now also U3.13 (PA7)
- net MSCLK: now also U3.11 (PA5)
- net NRST: now also U3.4 (NRST)
- net SWCLK: now also U3.24 (PA14)
- net SWDIO: now also U3.23 (PA13)
- net SW_BOOT0: now also SW1.2
- net TEST_LED: now also U3.28 (PB5)
- net USB_N: now also U3.21 (PA11)
- net USB_P: now also U3.22 (PA12)
Other:
- moved on the sheet: C10, C11, C12, C5, C6, C7, C8, C9, D4, FB1, J2, R10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
