File: Hardware/gyro_accel.kicad_sch (KiCad schematic)
At the start: 8 parts

Commit message: Restructure folders
Other:
- title: Robot Companion -> Robot Car Companion (DashiDaaa)
Changed lines of the file:
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@@
 	(paper "A4")
 	(title_block
-		(title "Robot Companion")
+		(title "Robot Car Companion (DashiDaaa)")
 		(date "2025-05-31")
 		(rev "B")
